File: Screw Driver/Screw Driver.kicad_pcb (KiCad board)
At the start: 2 copper layers, 56 x 95.5 mm, 47 parts, among them J1 V_Main, J10 MAIN TRIGGER, J11 V_OUT +, J12 V_OUT +, J2 Conn_01x05_Pin, J3 CW, J4 CCW, J5 OFF, J6 3v3, J7 POT_signal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

Commit message: Some routing done
Parts:
- C4: footprint Resistor_SMD:R_0603_1608Metric_Pad0.98x0.95mm_HandSolder -> Capacitor_SMD:C_0603_1608Metric_Pad1.08x0.95mm_HandSolder
- moved R12 31.5 mm to (132.5, 88.0), turned to 90 degrees
- moved R9 30.5 mm to (133.0, 85.0), turned to 0 degrees
- moved D1 28.6 mm to (117.9, 95.6)
- moved C8 28.5 mm to (122.5, 64.5)
- moved C9 28.5 mm to (122.5, 76.0)
- moved J1 28.5 mm to (128.1, 104.5)
- moved Q1 28.5 mm to (127.5, 87.0), turned to 180 degrees
- moved J3 9.84 mm to (163.5, 83.0)
- moved J4 9.02 mm to (163.5, 70.5)
- moved J5 7.56 mm to (163.5, 76.8)
- moved J6 4.50 mm to (169.0, 110.0)
- moved J7 4.50 mm to (169.0, 114.6)
- moved J8 4.50 mm to (169.0, 119.2)
- moved J10 0.91 mm to (160.5, 115.5)
- moved J11 0.65 mm to (142.7, 60.0)
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Connections:
- A1 pad 11: /DIAG_A_MCU -> unconnected-(A1-GPIO8-Pad11)
- A1 pad 12: /DIAG_B_MCU -> /MAIN_SW
- A1 pad 19: unconnected-(A1-GPIO14-Pad19) -> /IN_B
- A1 pad 20: /IN_B -> unconnected-(A1-GPIO15-Pad20)
- A1 pad 24: /MAIN_SW -> unconnected-(A1-GPIO18-Pad24)
- A1 pad 26: unconnected-(A1-GPIO20-Pad26) -> /IN_A
- A1 pad 5: /IN_A -> unconnected-(A1-GPIO3-Pad5)
- J3 pad 1: unconnected-(J3-Pin_1-Pad1) -> /CW
- J5 pad 1: unconnected-(J5-Pin_1-Pad1) -> GND
Routing:
- net /C_SENSE: track 0.00 -> 49.4 mm
- net /IN_A: track 0.00 -> 36.9 mm
- net /IN_B: track 0.00 -> 26.4 mm
- net /VCC: track 0.00 -> 25.6 mm, vias 0 -> 35
- net +5V: track 0.00 -> 21.1 mm
- net +12V: track 0.00 -> 19.3 mm
- net /DIAG_A_MCU: track 0.00 -> 18.7 mm
- net /PWM_MCU: track 0.00 -> 14.2 mm
- net /5V_SW: track 0.00 -> 8.41 mm
- net /DIAG_A: track 0.00 -> 6.29 mm
- net /MAIN_SW: track 0.00 -> 5.28 mm
- net /CS: track 0.00 -> 4.92 mm
- net Net-(Q1-G): track 0.00 -> 4.14 mm
- net /5V_FB: track 0.00 -> 2.58 mm
- net /5V_BST: track 0.00 -> 2.47 mm
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- added copper zone on F.Cu, net +12V
- added copper zone on B.Cu, net /OUT_A
- added copper zone on F.Cu, net /OUT_A
- added copper zone on B.Cu, net /OUT_B
- added copper zone on F.Cu, net /OUT_B
- added copper zone on F.Cu, net /VCC
Other:
- board text added: "3v3"
- board text added: "CCW"
- board text added: "GND"
- board text added: "Main SW"
- board text added: "POT SIGNAL"

Commit message: Some more routing done
Connections:
- A1 pad 31: /POT_SIG -> /C_SENSE
- A1 pad 32: /C_SENSE -> /POT_SIG
Routing:
- net /CS_DISABLE: track 0.00 -> 58.2 mm
- net /SWDIO: track 0.00 -> 55.7 mm, vias 0 -> 2
- net /SWCLK: track 0.00 -> 49.7 mm, vias 0 -> 1
- net /CCW: track 0.00 -> 42.7 mm, vias 0 -> 2
- net +3V3: track 0.00 -> 36.9 mm, vias 0 -> 1
- net /POT_SIG: track 0.00 -> 36.7 mm
- net +5V: track 21.1 -> 48.1 mm, vias 0 -> 2
- net /CW: track 0.00 -> 25.2 mm, vias 0 -> 1
- net +12V: track 19.3 -> 42.5 mm, vias 0 -> 2
- net /DIAG_B_MCU: track 0.00 -> 20.0 mm
- net /CP: track 0.00 -> 18.9 mm, vias 0 -> 2
- net /PWM: track 0.00 -> 8.43 mm, vias 0 -> 2
- net /DEBUG_TX: track 0.00 -> 5.13 mm
- net /DEBUG_RX: track 0.00 -> 5.02 mm
- net /C_SENSE: track 49.4 -> 46.8 mm
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- added copper zone on B.Cu, net /VCC

Commit message: Routing fully done
Parts:
- moved R1 0.25 mm to (144.2, 83.4)
Routing:
- net +5V: track 48.1 -> 106.3 mm, vias 2 -> 3
- net /VCC: track 27.7 -> 46.1 mm
- net /DIAG_B: track 0.00 -> 15.3 mm, vias 0 -> 2
- net GND: track 0.01 -> 15.2 mm, vias 2 -> 12
- net /CS_DISABLE: track 58.2 -> 44.3 mm, vias 0 -> 2
- net +3V3: track 36.9 -> 45.4 mm
- net /5V_FB: track 2.58 -> 9.15 mm
- net /PWM: track 8.43 -> 10.9 mm
- net /IN_A: track 36.9 -> 37.7 mm
Other:
- board text added: "12V"
- board text added: "CW"
- board text added: "POT SIG"
- board text removed: "POT SIGNAL"

Commit message: Improved Layout
Routing:
- net +12V: track 42.6 -> 23.3 mm
- net /VCC: track 46.1 -> 41.5 mm
Changed lines of the file:
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@@
 		)
 		(fp_text user "USB Cable"
-			(at 0 -38.735 180)
+			(at 0 -30.31 0)
 			(unlocked yes)
 			(layer "Cmts.User")
@@
 		)
 		(fp_text user "Keep Out"
-			(at 0 -36.195 180)
+			(at 0 -32.85 0)
 			(unlocked yes)
 			(layer "Cmts.User")
@@
 	)
 	(gr_text "3v3"
-		(at 165.957146 109.945353 0)
+		(at 164.75 110 0)
 		(layer "F.SilkS")
 		(effects
 			(font
+				(face "JetBrains Mono NL SemiBold")
 				(size 1 1)
 				(thickness 0.15)
 			)
 		)
+		(render_cache "3v3" 0
+			(polygon
+				(pts
+					(xy 163.898264 110.428982) (xy 163.825121 110.423485) (xy 163.763393 110.407991) (xy 163.711104 110.383435)
+					(xy 163.666722 110.34997) (xy 163.630337 110.307831) (xy 163.604134 110.25896) (xy 163.587829 110.202034)
+					(xy 163.582092 110.135219) (xy 163.733217 110.135219) (xy 163.738556 110.182754) (xy 163.75359 110.221235)
+					(xy 163.777975 110.2527) (xy 163.810251 110.276186) (xy 163.850102 110.290822) (xy 163.899669 110.296053)
+					(xy 163.949235 110.290822) (xy 163.989087 110.276186) (xy 164.021363 110.2527) (xy 164.045783 110.221231)
+					(xy 164.060836 110.182749) (xy 164.066181 110.135219) (xy 164.066181 110.062435) (xy 164.060767 110.013013)
+					(xy 164.045651 109.973676) (xy 164.021363 109.942145) (xy 163.989082 109.918624) (xy 163.949231 109.903968)
+					(xy 163.899669 109.898731) (xy 163.780783 109.898731) (xy 163.780783 109.772824) (xy 164.022828 109.528032)
+					(xy 163.614271 109.528032) (xy 163.614271 109.393698) (xy 164.190684 109.393698) (xy 164.190684 109.526627)
+					(xy 163.950044 109.770076) (xy 164.011257 109.781035) (xy 164.063401 109.799929) (xy 164.107916 109.826312)
+					(xy 164.145865 109.860324) (xy 164.17653 109.901038) (xy 164.198682 109.947308) (xy 164.212434 110.00018)
+					(xy 164.217245 110.061031) (xy 164.217245 110.135219) (xy 164.21143 110.201944) (xy 164.194888 110.258839)
+					(xy 164.168262 110.307742) (xy 164.131211 110.34997) (xy 164.086183 110.383479) (xy 164.03341 110.408036)
+					(xy 163.971407 110.423505)
+				)
+			)
+			(polygon
+				(pts
+					(xy 164.653585 110.415) (xy 164.393345 109.645512) (xy 164.552835 109.645512) (xy 164.710921 110.137967)
+					(xy 164.736078 110.224063) (xy 164.75287 110.29471) (xy 164.767586 110.224063) (xy 164.790667 110.137967)
+					(xy 164.947348 109.645512) (xy 165.106839 109.645512) (xy 164.848003 110.415)
+				)
+			)
+			(polygon
+				(pts
+					(xy 165.576701 110.428982) (xy 165.503558 110.423485) (xy 165.44183 110.407991) (xy 165.389541 110.383435)
+					(xy 165.345159 110.34997) (xy 165.308773 110.307831) (xy 165.282571 110.25896) (xy 165.266266 110.202034)
+					(xy 165.260529 110.135219) (xy 165.411654 110.135219) (xy 165.416993 110.182754) (xy 165.432027 110.221235)
+					(xy 165.456412 110.2527) (xy 165.488687 110.276186) (xy 165.528539 110.290822) (xy 165.578106 110.296053)
+					(xy 165.627672 110.290822) (xy 165.667524 110.276186) (xy 165.6998 110.2527) (xy 165.72422 110.221231)
+					(xy 165.739273 110.182749) (xy 165.744618 110.135219) (xy 165.744618 110.062435) (xy 165.739204 110.013013)
+					(xy 165.724088 109.973676) (xy 165.6998 109.942145) (xy 165.667519 109.918624) (xy 165.627668 109.903968)
+					(xy 165.578106 109.898731) (xy 165.45922 109.898731) (xy 165.45922 109.772824) (xy 165.701265 109.528032)
+					(xy 165.292708 109.528032) (xy 165.292708 109.393698) (xy 165.869121 109.393698) (xy 165.869121 109.526627)
+					(xy 165.628481 109.770076) (xy 165.689694 109.781035) (xy 165.741838 109.799929) (xy 165.786353 109.826312)
+					(xy 165.824302 109.860324) (xy 165.854967 109.901038) (xy 165.877118 109.947308) (xy 165.890871 110.00018)
+					(xy 165.895682 110.061031) (xy 165.895682 110.135219) (xy 165.889866 110.201944) (xy 165.873325 110.258839)
+					(xy 165.846699 110.307742) (xy 165.809648 110.34997) (xy 165.76462 110.383479) (xy 165.711847 110.408036)
+					(xy 165.649844 110.423505)
+				)
+			)
+		)
 	)
 	(gr_text "POT\nSIG"
@@
 	)
 	(via
-		(at 148.5 83)
+		(at 148.25 84)
 		(size 0.5)
 		(drill 0.3)
@@
 	)
 	(segment
-		(start 130.261409 91.698673)
-		(end 130.24725 91.684514)
-		(width 1)
-		(layer "F.Cu")
-		(net 27)
-	)
-	(segment
-		(start 130.24725 91.684514)
-		(end 130.24725 86.365)
-		(width 1)
-		(layer "F.Cu")
-		(net 27)
-	)
-	(segment
-		(start 126.38704 95.573042)
-		(end 130.261409 91.698673)
-		(width 1)
-		(layer "F.Cu")
-		(net 27)
-	)
-	(segment
-		(start 117.938914 95.573042)
-		(end 126.38704 95.573042)
-		(width 1)
-		(layer "F.Cu")
-		(net 27)
-	)
-	(segment
 		(start 148.5 78.125)
 		(end 148.5 79)
@@
 	)
 	(segment
-		(start 126.755 86.755)
-		(end 123.5 83.5)
-		(width 1)
-		(layer "F.Cu")
-		(net 43)
-	)
-	(segment
 		(start 162.225 98.0875)
 		(end 162.6375 98.5)
@@
 			)
 		)
+	)
+	(zone
+		(net 27)
+		(net_name "+12V")
+		(layer "F.Cu")
+		(hatch edge 0.5)
+		(priority 11)
+		(connect_pads yes
+			(clearance 0.5)
+		)
+		(min_thickness 0.25)
+		(filled_areas_thickness no)
+		(fill yes
+			(thermal_gap 0.5)
+			(thermal_bridge_width 0.5)
+		)
+		(polygon
+			(pts
+				(xy 129.5 85.75) (xy 129.5 91) (xy 116 91) (xy 116 109) (xy 124.5 109) (xy 124.5 98.25) (xy 131.25 98.25)
+				(xy 131.25 85.75)
+			)
+		)
