File: DRV8701-ESD/DRV8701-ESD.kicad_sch (KiCad schematic)
At the start: 55 parts

Commit message: Finalized few components
Parts:
- removed C? (x2): 4.7u, Capacitor_SMD:C_1206_3216Metric_Pad1.33x1.80mm_HandSolder, symbol Device:C_Small
- removed C?: 470u, Capacitor_THT:C_Radial_D10.0mm_H20.0mm_P5.00mm, symbol Device:C_Small
- removed C?: 10u, Capacitor_SMD:C_0603_1608Metric_Pad1.08x0.95mm_HandSolder, symbol Device:C_Small
- removed Q?: NVMFS5C628NLET1G, Package_SO:ONSemi_SO-8FL_488AA, symbol Mosfet_PWR:NTMFS2D5N08XT1G
- removed R?: 100k, Resistor_SMD:R_0603_1608Metric_Pad0.98x0.95mm_HandSolder, symbol Device:R
- removed R?: 10, Resistor_SMD:R_0603_1608Metric_Pad0.98x0.95mm_HandSolder, symbol Device:R
- removed R?: 47k, Resistor_SMD:R_0603_1608Metric_Pad0.98x0.95mm_HandSolder, symbol Device:R
- removed R?: 13.7k, Capacitor_SMD:C_0603_1608Metric_Pad1.08x0.95mm_HandSolder, symbol Device:R
- added C10, C11, C12, C13: 100n, Capacitor_SMD:C_0603_1608Metric_Pad1.08x0.95mm_HandSolder, symbol Device:C_Small
- added C14, C3, C6, C7: 10u, Capacitor_SMD:C_1206_3216Metric_Pad1.33x1.80mm_HandSolder, symbol Device:C_Small
- added C19: 470u, Capacitor_THT:C_Radial_D10.0mm_H20.0mm_P5.00mm, symbol Device:C_Small
- added D2, D3: RBR10N, Package_TO_SOT_SMD:TO-263-2, symbol Device:D_Schottky
- added NT1, NT2: NetTie_2, Net_Ties:NetTie_0.2mm_SMD, symbol Device:NetTie_2
- added R1, R10, R2, R9: 100k, Resistor_SMD:R_0603_1608Metric_Pad0.98x0.95mm_HandSolder, symbol Device:R
- C20: renamed from C?; MFP B41859C7477M8 -> EEU-FM1V471
- D4: renamed from D?; value 1.5KE18A -> SMBJ18A; footprint Diode_THT:D_DO-201AE_P15.24mm_Horizontal -> Diode_SMD:D_SMA-SMB_Universal_Handsoldering
- L1: renamed from L?; footprint Inductor_SMD:L_Changjiang_FXL0420 -> Inductor_SMD:L_6.3x6.3_H3
- U1: renamed from U?; footprint RGE0024F -> (none)
- gave numbers to parts that had none: 42
Connections:
- net 5V_FB is gone; now on net +5V: U2.1 (FB)
- net VM is gone; now on net VCC: C4.1
- net +12V: now also D2.2 (A), D3.2 (A)
- net GH1: now also R1.1
- net GH2: now also R9.1
- net GL1: now also R2.1
- net GL2: now also R10.1
- net GND: now also U1.5 (GND), C10.1, C11.1, C12.1, C13.1, C14.1, C19.2, C3.1, C6.1, C7.1, NT2.2, R1.2, R10.2, R2.2, R9.2; no longer U1.20 (SN)
- net SO: now also A1.31 (GPIO26_ADC0)
- net SP: now also NT1.1; no longer Q2.1 (S), Q2.2 (S), Q2.3 (S), Q4.1 (S), Q4.2 (S), Q4.3 (S), R7.1
- net VCC: now also C10.2, C11.2, C12.2, C13.2, C14.2, C19.1, C3.2, C6.2, C7.2, D2.1 (K), D3.1 (K)
- net nFAULT: now also A1.25 (GPIO19)
- net nSLEEP: now also A1.21 (GPIO16)
- net PH_DIR: now reaches A1.22 (GPIO17)
- net PH_DIR: now also U1.15 (PH_IN1)
- net EN_PWM: now reaches A1.26 (GPIO20)
- net EN_PWM: now also U1.14 (EN_IN2)
- new net SN: NT2.1, U1.20 (SN)
- new net SP_TOP: NT1.2, Q2.1 (S), Q2.2 (S), Q2.3 (S), Q4.1 (S), Q4.2 (S), Q4.3 (S), R7.1
- no-connect marks 19 -> 21
Other:
- note removed: "REVERSE VOLTAGE PROTECTION"
- moved on the sheet: A1, C1, C15, C16, C17, C18, C2, C20, C4, C5, C8, C9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

Commit message: Some Routing done
Parts:
- removed D2, D3: RBR10N, Package_TO_SOT_SMD:TO-263-2, symbol Device:D_Schottky
- added D2, D3: RBR10N, Package_TO_SOT_SMD:TO-263-2, symbol Device:D_Schottky_AKA
- C16, C17: footprint Capacitor_SMD:C_0805_2012Metric_Pad1.18x1.45mm_HandSolder -> Capacitor_SMD:C_1210_3225Metric_Pad1.33x2.70mm_HandSolder
- R7: footprint (none) -> Resistor_SMD:R_2512_6332Metric_Pad1.40x3.35mm_HandSolder
- U1: footprint (none) -> DRV8701:RGE0024F_NV
Connections:
- net +12V: now also D2.1 (A), D2.3 (A), D3.1 (A), D3.3 (A)
- net VCC: now also D2.2 (K), D3.2 (K)
Changed lines of the file:
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@@
 	)
 	(junction
-		(at 99.06 243.84)
+		(at 335.28 147.32)
 		(diameter 0)
 		(color 0 0 0 0)
 	)
 	(junction
-		(at 80.01 189.23)
+		(at 99.06 243.84)
 		(diameter 0)
 		(color 0 0 0 0)
 	)
 	(junction
-		(at 69.85 251.46)
+		(at 80.01 189.23)
 		(diameter 0)
 		(color 0 0 0 0)
 	)
 	(junction
-		(at 346.71 147.32)
+		(at 69.85 251.46)
 		(diameter 0)
 		(color 0 0 0 0)
@@
 	)
 	(junction
+		(at 346.71 147.32)
+		(diameter 0)
+		(color 0 0 0 0)
+	)
+	(junction
 		(at 278.13 161.29)
 		(diameter 0)
@@
 	)
 	(junction
+		(at 334.01 157.48)
+		(diameter 0)
+		(color 0 0 0 0)
+	)
+	(junction
 		(at 330.2 102.87)
 		(diameter 0)
@@
 	(wire
 		(pts
+			(xy 344.17 147.32) (xy 346.71 147.32)
+		)
+		(stroke
+			(width 0)
+			(type default)
+		)
+	)
+	(wire
+		(pts
 			(xy 278.13 161.29) (xy 278.13 162.56)
 		)
@@
 	(wire
 		(pts
-			(xy 342.9 152.4) (xy 346.71 152.4)
+			(xy 342.9 157.48) (xy 346.71 157.48)
 		)
 		(stroke
@@
 	(wire
 		(pts
-			(xy 335.28 152.4) (xy 331.47 152.4)
+			(xy 251.46 144.78) (xy 259.08 144.78)
 		)
 		(stroke
@@
 	(wire
 		(pts
-			(xy 251.46 144.78) (xy 259.08 144.78)
+			(xy 57.15 29.21) (xy 63.5 29.21)
 		)
 		(stroke
@@
 	(wire
 		(pts
-			(xy 57.15 29.21) (xy 63.5 29.21)
+			(xy 331.47 157.48) (xy 334.01 157.48)
 		)
 		(stroke
@@
 	(wire
 		(pts
-			(xy 331.47 152.4) (xy 331.47 147.32)
+			(xy 331.47 157.48) (xy 331.47 147.32)
 		)
 		(stroke
@@
 	(wire
 		(pts
+			(xy 334.01 157.48) (xy 334.01 160.02)
+		)
+		(stroke
+			(width 0)
+			(type default)
+		)
+	)
+	(wire
+		(pts
 			(xy 111.76 39.37) (xy 104.14 39.37)
 		)
@@
 	(wire
 		(pts
-			(xy 346.71 152.4) (xy 346.71 147.32)
+			(xy 346.71 157.48) (xy 346.71 147.32)
 		)
 		(stroke
@@
 	(wire
 		(pts
+			(xy 335.28 147.32) (xy 335.28 149.86)
+		)
+		(stroke
+			(width 0)
+			(type default)
+		)
+	)
+	(wire
+		(pts
 			(xy 327.66 102.87) (xy 327.66 105.41)
 		)
@@
 	(wire
 		(pts
-			(xy 346.71 147.32) (xy 342.9 147.32)
-		)
-		(stroke
-			(width 0)
-			(type default)
-		)
-	)
-	(wire
-		(pts
 			(xy 203.2 50.8) (xy 218.44 50.8)
 		)
@@
 			)
 		)
-		(property "Footprint" ""
+		(property "Footprint" "Resistor_SMD:R_2512_6332Metric_Pad1.40x3.35mm_HandSolder"
 			(at 105.41 222.25 0)
 			(effects
@@
 			)
 		)
-		(property "Footprint" ""
+		(property "Footprint" "DRV8701:RGE0024F_NV"
 			(at 83.82 57.15 0)
 			(effects
@@
 	)
 	(symbol
-		(lib_id "Device:D_Schottky")
-		(at 339.09 147.32 180)
-		(unit 1)
-		(exclude_from_sim no)
-		(in_bom yes)
-		(on_board yes)
-		(dnp no)
-		(fields_autoplaced yes)
-		(property "Reference" "D2"
-			(at 339.4075 140.97 0)
-			(effects
-				(font
-					(size 1.27 1.27)
-				)
-			)
-		)
-		(property "Value" "RBR10N"
-			(at 339.4075 143.51 0)
-			(effects
-				(font
-					(size 1.27 1.27)
-				)
-			)
-		)
-		(property "Footprint" "Package_TO_SOT_SMD:TO-263-2"
-			(at 339.09 147.32 0)
-			(effects
-				(font
-					(size 1.27 1.27)
-				)
-				(hide yes)
-			)
-		)
-		(property "Datasheet" "https://prod-parts-data.s3.amazonaws.com/RBR10NS40AFHTL/datasheet/1_RBR10NS40AFHTL-Rohm-datasheet-142143708.pdf"
-			(at 339.09 147.32 0)
-			(effects
-				(font
-					(size 1.27 1.27)
-				)
-				(hide yes)
-			)
-		)
-		(property "Description" "RBR10NS40AFHTL"
-			(at 339.09 147.32 0)
-			(effects
-				(font
-					(size 1.27 1.27)
-				)
-				(hide yes)
-			)
-		)
-		(pin "2"
-		)
-		(pin "1"
-		)
-		(instances
-			(project ""
-				(path "/b24bf440-a013-4035-96b7-c33cc728982a"
-					(reference "D2")
-					(unit 1)
-				)
-			)
-		)
-	)
-	(symbol
 		(lib_id "Connector:Conn_01x01_Pin")
 		(at 320.04 72.39 0)
@@
 		(dnp no)
 		(property "Reference" "C17"
-			(at 273.558 160.274 90)
+			(at 274.574 160.274 90)
 			(effects
 				(font
@@
 			)
 		)
-		(property "Footprint" "Capacitor_SMD:C_0805_2012Metric_Pad1.18x1.45mm_HandSolder"
+		(property "Footprint" "Capacitor_SMD:C_1210_3225Metric_Pad1.33x2.70mm_HandSolder"
 			(at 270.51 161.29 0)
 			(effects
@@
 		(dnp no)
 		(property "Reference" "C16"
-			(at 273.558 153.924 90)
+			(at 274.574 153.924 90)
 			(effects
 				(font
@@
 			)
 		)
-		(property "Footprint" "Capacitor_SMD:C_0805_2012Metric_Pad1.18x1.45mm_HandSolder"
+		(property "Footprint" "Capacitor_SMD:C_1210_3225Metric_Pad1.33x2.70mm_HandSolder"
 			(at 270.51 154.94 0)
 			(effects
@@
 	)
 	(symbol
+		(lib_id "Device:D_Schottky_AKA")
+		(at 339.09 157.48 180)
+		(unit 1)
+		(exclude_from_sim no)
+		(in_bom yes)
+		(on_board yes)
+		(dnp no)
+		(property "Reference" "D2"
+			(at 339.09 159.766 0)
+			(effects
+				(font
+					(size 1.27 1.27)
+				)
+			)
+		)
+		(property "Value" "RBR10N"
+			(at 339.09 155.194 0)
+			(effects
+				(font
+					(size 1.27 1.27)
+				)
+			)
+		)
+		(property "Footprint" "Package_TO_SOT_SMD:TO-263-2"
+			(at 339.09 157.48 0)
+			(effects
+				(font
+					(size 1.27 1.27)
+				)
+				(hide yes)
+			)
+		)
+		(property "Datasheet" "https://prod-parts-data.s3.amazonaws.com/RBR10NS40AFHTL/datasheet/1_RBR10NS40AFHTL-Rohm-datasheet-142143708.pdf"
+			(at 339.09 157.48 0)
+			(effects
+				(font
+					(size 1.27 1.27)
+				)
+				(hide yes)
+			)
+		)
+		(property "Description" "RBR10NS40AFHTL"
+			(at 339.09 157.48 0)
+			(effects
+				(font
+					(size 1.27 1.27)
+				)
+				(hide yes)
+			)
+		)
+		(pin "3"
+		)
+		(pin "1"
+		)
+		(pin "2"
+		)
+		(instances
+			(project "DRV8701-ESD"
+				(path "/b24bf440-a013-4035-96b7-c33cc728982a"
+					(reference "D2")
+					(unit 1)
+				)
+			)
+		)
+	)
+	(symbol
 		(lib_id "Mechanical:MountingHole_Pad")
 		(at 369.57 74.93 0)
@@
 	)
 	(symbol
+		(lib_id "Device:D_Schottky_AKA")
+		(at 340.36 147.32 180)
+		(unit 1)
+		(exclude_from_sim no)
+		(in_bom yes)
+		(on_board yes)
+		(dnp no)
+		(property "Reference" "D3"
+			(at 340.36 150.114 0)
+			(effects
+				(font
+					(size 1.27 1.27)
+				)
+			)
+		)
+		(property "Value" "RBR10N"
+			(at 342.138 144.272 0)
+			(effects
+				(font
+					(size 1.27 1.27)
+				)
+			)
+		)
+		(property "Footprint" "Package_TO_SOT_SMD:TO-263-2"
+			(at 340.36 147.32 0)
+			(effects
+				(font
+					(size 1.27 1.27)
+				)
+				(hide yes)
+			)
+		)
+		(property "Datasheet" "https://prod-parts-data.s3.amazonaws.com/RBR10NS40AFHTL/datasheet/1_RBR10NS40AFHTL-Rohm-datasheet-142143708.pdf"
+			(at 340.36 147.32 0)
+			(effects
+				(font
+					(size 1.27 1.27)
+				)
+				(hide yes)
+			)
+		)
+		(property "Description" "RBR10NS40AFHTL"
+			(at 340.36 147.32 0)
+			(effects
+				(font
+					(size 1.27 1.27)
+				)
+				(hide yes)
+			)
+		)
+		(pin "3"
+		)
+		(pin "1"
+		)
+		(pin "2"
+		)
+		(instances
+			(project ""
+				(path "/b24bf440-a013-4035-96b7-c33cc728982a"
+					(reference "D3")
+					(unit 1)
+				)
+			)
+		)
+	)
+	(symbol
 		(lib_id "power:PWR_FLAG")
 		(at 137.16 21.59 180)
@@
 					(unit 1)
 				)
-			)
-		)
-	)
-	(symbol
-		(lib_id "Device:D_Schottky")
-		(at 339.09 152.4 180)
-		(unit 1)
-		(exclude_from_sim no)
-		(in_bom yes)
-		(on_board yes)
-		(dnp no)
-		(property "Reference" "D3"
-			(at 339.598 154.686 0)
-			(effects
-				(font
-					(size 1.27 1.27)
-				)
-			)
-		)
-		(property "Value" "RBR10N"
-			(at 339.598 157.226 0)
-			(effects
-				(font
-					(size 1.27 1.27)
-				)
-			)
-		)
-		(property "Footprint" "Package_TO_SOT_SMD:TO-263-2"
-			(at 339.09 152.4 0)
-			(effects
-				(font
-					(size 1.27 1.27)
-				)
-				(hide yes)
-			)
-		)
-		(property "Datasheet" "https://prod-parts-data.s3.amazonaws.com/RBR10NS40AFHTL/datasheet/1_RBR10NS40AFHTL-Rohm-datasheet-142143708.pdf"
-			(at 339.09 152.4 0)
-			(effects
-				(font
-					(size 1.27 1.27)
-				)
-				(hide yes)
-			)
-		)
-		(property "Description" "RBR10NS40AFHTL"
-			(at 339.09 152.4 0)
-			(effects
-				(font
-					(size 1.27 1.27)
-				)
-				(hide yes)
-			)
-		)
-		(pin "2"
-		)
-		(pin "1"
-		)
-		(instances
-			(project "DRV8701-ESD"
-				(path "/b24bf440-a013-4035-96b7-c33cc728982a"
-					(reference "D3")
-					(unit 1)
-				)
