File: DRV8701-ESD/DRV8701-ESD.kicad_sch (KiCad schematic)
At the start: 63 parts, among them J1 V_Main, J10 POT_signal, J11 GND, J12 Conn_01x05_Pin, J2 V_OUT -, J3 V_OUT +, J4 CW, J5 OFF, J6 CCW, J7 MAIN TRIGGER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

Commit message: Added PMOS, Changed VREF to 3v3, Added 5->3v3 LDO, Placed components tentatively. Yet to review.
Parts:
- removed D2, D3: RBR10N, Package_TO_SOT_SMD:TO-263-2, symbol Device:D_Schottky_AKA
- added C21: 10u, Capacitor_SMD:C_1206_3216Metric_Pad1.33x1.80mm_HandSolder, symbol Device:C_Small
- added C22: 22u, Capacitor_SMD:C_1210_3225Metric_Pad1.33x2.70mm_HandSolder, symbol Device:C_Small
- added D2: BZT52C12, Diode_SMD:D_SOD-123F, symbol Diode:BZT52Bxx
- added Q5: IPB80P04P4L08ATMA2, Package_TO_SOT_SMD:TO-263-2, symbol TJ40S04M3L:TJ40S04M3L,LXHQ
- added R14: 100k, Resistor_SMD:R_0603_1608Metric_Pad0.98x0.95mm_HandSolder, symbol Device:R
- added R15: 33k, Resistor_SMD:R_0603_1608Metric_Pad0.98x0.95mm_HandSolder, symbol Device:R
- added U3: AZ1117CH2-3.3, Package_TO_SOT_SMD:SOT-223-3_TabPin2, symbol Regulator_Linear:AZ1117CH2-3.3
- R5: now not fitted
Connections:
- net +12V: now also D2.1 (K), Q5.3 (S); no longer D4.1 (A1)
- net +3V3: now also U1.6 (VREF), C22.2, U3.3 (OUT); no longer A1.36 (3V3)
- net +5V: now also C21.1, U3.1 (IN)
- net AVDD: now also R15.1; no longer U1.6 (VREF)
- net GND: now also C21.2, C22.1, R14.2, U3.2 (GND)
- net IDRIVE: now also R15.2
- net VCC: now also D4.1 (A1), Q5.2 (D)
- new net: D2.2 (A), Q5.1 (G), R14.1
- no-connect marks 21 -> 22

Commit message: Some more stuff added
Parts:
- added C23: 100n, Capacitor_SMD:C_0603_1608Metric_Pad1.08x0.95mm_HandSolder, symbol Device:C_Small
- added R16: 10k, Resistor_SMD:R_0603_1608Metric_Pad0.98x0.95mm_HandSolder, symbol Device:R
- added R17: 20k, Resistor_SMD:R_0603_1608Metric_Pad0.98x0.95mm_HandSolder, symbol Device:R
- added R18, R19: 100k, Resistor_SMD:R_0603_1608Metric_Pad0.98x0.95mm_HandSolder, symbol Device:R
Connections:
- net +3V3: now also R18.1
- net GND: now also C23.1, R17.1, R19.2
- net POT_SIG: now also R18.2, R19.1
- net SO: now also C23.2, R16.2; no longer A1.31 (GPIO26_ADC0)
- new net SO_MCU: A1.31 (GPIO26_ADC0), R16.1, R17.2

Commit message: Changes done after review
Parts:
- removed C23: 100n, Capacitor_SMD:C_0603_1608Metric_Pad1.08x0.95mm_HandSolder, symbol Device:C_Small
- L1: footprint Inductor_SMD:L_6.3x6.3_H3 -> Inductor_SMD_Custom:L_SMD_6mmx6mm
Connections:
- net +3V3: no longer U1.6 (VREF)
- net AVDD: now also U1.6 (VREF)
Other:
- note added: "RVP"
