File: DRV8701-ESD/DRV8701-ESD.kicad_pcb (KiCad board)
At the start: 4 copper layers, 55 x 95 mm, 78 parts, among them J1 V_Main, J10 POT_signal, J11 GND, J12 Conn_01x05_Pin, J13 CW, J14 CW, J15 CW, J17 CW, J18 CW, J19 CW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

Commit message: Made some final changes, ordered.
Parts:
- added G***: LOGO, komi:komi_1, F.Cu at (165.7, 50.5)
- added G***: LOGO, komi:frieren, B.Cu at (166.5, 137.2)
- added G***: LOGO, komi:komi_1, B.Cu at (135.5, 50.2)
- moved C16 0.32 mm to (136.2, 102.2)
- moved L1 0.17 mm to (135.6, 93.1)
Routing:
- net GND: track 22.9 -> 38.8 mm, vias 59 -> 73
Other:
- outline, holes or cut-outs redrawn
