File: Screw Driver/DRV8701-ESD/DRV8701-ESD.kicad_pcb (KiCad board)
At the start: 4 copper layers, 55 x 95 mm, 79 parts, among them J1 V_Main, J10 POT_signal, J11 GND, J12 Conn_01x05_Pin, J13 CW, J14 CW, J15 CW, J16 Conn_01x05_Pin, J17 CW, J18 CW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

Commit message: Made improvements.
Parts:
- removed J16: Conn_01x05_Pin, Connector_Molex:Molex_PicoBlade_53398-0571_1x05-1MP_P1.25mm_Vertical
- moved R13 15.3 mm to (129.2, 105.8), turned to -90 degrees
- moved C17 13.2 mm to (136.5, 92.2), turned to 180 degrees
- moved D1 12.1 mm to (132.2, 105.7), turned to 90 degrees
- moved L1 11.9 mm to (135.5, 93.0), turned to 180 degrees
- moved C18 8.14 mm to (130.2, 94.5)
- moved C15 6.47 mm to (126.5, 97.2), turned to 90 degrees
- moved C14 6.17 mm to (129.0, 100.2), turned to 180 degrees
- moved U2 3.81 mm to (129.6, 97.2), turned to 0 degrees
- moved C16 3.42 mm to (136.5, 102.0), turned to 180 degrees
Routing:
- net +5V: track 67.8 -> 38.3 mm, vias 30 -> 58
- net /VCC: track 42.6 -> 26.9 mm, vias 194 -> 188
- net /5V_SW: track 11.2 -> 0.00 mm
- net MOTOR+: track 33.1 -> 25.7 mm, vias 77 -> 101
- net MOTOR-: track 30.0 -> 23.0 mm, vias 83 -> 107
- net /DEBUG_RX: track 15.6 -> 14.2 mm
- net /SWDIO: track 46.4 -> 45.0 mm
- net /SWCLK: track 43.1 -> 41.7 mm
- net /DEBUG_TX: track 16.7 -> 15.3 mm
- net Net-(D1-K): track 1.96 -> 2.98 mm
- net /5V_BST: track 1.85 -> 2.36 mm
- net GND: track 22.2 -> 21.7 mm, vias 38 -> 58
- net /SP_TOP: vias 9 -> 28
- added copper zone on F.Cu, net /5V_SW
- added copper zone on B.Cu, net /SP_TOP
Other:
- outline, holes or cut-outs redrawn
- board text added: "BUCK"
- board text added: "RVP-PMOS"
