File: Screw Driver/DRV8701-ESD/DRV8701-ESD.kicad_sch (KiCad schematic)
At the start: 79 parts, among them J1 V_Main, J10 POT_signal, J11 GND, J12 Conn_01x05_Pin, J13 CW, J14 CW, J15 CW, J16 Conn_01x05_Pin, J17 CW, J18 CW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

Commit message: Made improvements.
Parts:
- removed J16: Conn_01x05_Pin, Molex_PicoBlade_53398-0571_1x05-1MP_P1.25mm_Vertical, symbol Connector:Conn_01x05_Pin
Changed lines of the file:
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@@
 		)
 	)
-	(label "SWCLK"
-		(at 397.51 109.22 0)
-		(effects
-			(font
-				(size 1.27 1.27)
-			)
-			(justify left bottom)
-		)
-	)
 	(label "5V_BST"
 		(at 292.1 147.32 180)
@@
 		)
 	)
-	(label "DEBUG_RX"
-		(at 397.51 106.68 0)
-		(effects
-			(font
-				(size 1.27 1.27)
-			)
-			(justify left bottom)
-		)
-	)
 	(label "MAIN_SW"
 		(at 320.04 60.96 0)
@@
 		)
 	)
-	(label "DEBUG_TX"
-		(at 397.51 104.14 0)
-		(effects
-			(font
-				(size 1.27 1.27)
-			)
-			(justify left bottom)
-		)
-	)
 	(label "GL2"
 		(at 114.3 196.85 0)
@@
 		)
 	)
-	(label "SWDIO"
-		(at 397.51 111.76 0)
-		(effects
-			(font
-				(size 1.27 1.27)
-			)
-			(justify left bottom)
-		)
-	)
 	(label "SP_TOP"
 		(at 105.41 218.44 0)
@@
 	)
 	(symbol
-		(lib_id "Connector:Conn_01x05_Pin")
-		(at 392.43 109.22 0)
-		(mirror x)
-		(unit 1)
-		(exclude_from_sim no)
-		(in_bom yes)
-		(on_board yes)
-		(dnp no)
-		(property "Reference" "J16"
-			(at 392.6373 115.8115 0)
-			(effects
-				(font
-					(size 1.27 1.27)
-				)
-			)
-		)
-		(property "Value" "Conn_01x05_Pin"
-			(at 398.018 99.822 0)
-			(effects
-				(font
-					(size 1.27 1.27)
-				)
-			)
-		)
-		(property "Footprint" "Molex_PicoBlade_53398-0571_1x05-1MP_P1.25mm_Vertical"
-			(at 392.43 109.22 0)
-			(effects
-				(font
-					(size 1.27 1.27)
-				)
-				(hide yes)
-			)
-		)
-		(property "Datasheet" "~"
-			(at 392.43 109.22 0)
-			(effects
-				(font
-					(size 1.27 1.27)
-				)
-				(hide yes)
-			)
-		)
-		(property "Description" "Generic connector, single row, 01x05, script generated"
-			(at 392.43 109.22 0)
-			(effects
-				(font
-					(size 1.27 1.27)
-				)
-				(hide yes)
-			)
-		)
-		(pin "2"
-		)
-		(pin "5"
-		)
-		(pin "4"
-		)
-		(pin "3"
-		)
-		(pin "1"
-		)
-		(instances
-			(project "DRV8701-ESD"
-				(path "/b24bf440-a013-4035-96b7-c33cc728982a"
-					(reference "J16")
-					(unit 1)
-				)
-			)
-		)
-	)
-	(symbol
 		(lib_id "Device:C_Small")
 		(at 231.14 179.07 90)
@@
 					(unit 1)
 				)
-			)
-		)
-	)
-	(symbol
-		(lib_id "power:GND")
-		(at 397.51 114.3 0)
-		(unit 1)
-		(exclude_from_sim no)
-		(in_bom yes)
-		(on_board yes)
-		(dnp no)
-		(fields_autoplaced yes)
-		(property "Reference" "#PWR015"
-			(at 397.51 120.65 0)
-			(effects
-				(font
-					(size 1.27 1.27)
-				)
-				(hide yes)
-			)
-		)
-		(property "Value" "GND"
-			(at 397.51 119.38 0)
-			(effects
-				(font
-					(size 1.27 1.27)
-				)
-				(hide yes)
-			)
-		)
-		(property "Footprint" ""
-			(at 397.51 114.3 0)
-			(effects
-				(font
-					(size 1.27 1.27)
-				)
-				(hide yes)
-			)
-		)
-		(property "Datasheet" ""
-			(at 397.51 114.3 0)
-			(effects
-				(font
-					(size 1.27 1.27)
-				)
-				(hide yes)
-			)
-		)
-		(property "Description" "Power symbol creates a global label with name \"GND\" , ground"
-			(at 397.51 114.3 0)
-			(effects
-				(font
-					(size 1.27 1.27)
-				)
-				(hide yes)
-			)
-		)
-		(pin "1"
-		)
-		(instances
-			(project "DRV8701-ESD"
-				(path "/b24bf440-a013-4035-96b7-c33cc728982a"
-					(reference "#PWR015")
-					(unit 1)
-				)
